Commit message: simplified RFL model
without Z axis mimicking joint

File: src/rfl/urdf/cart_macro.xacro (robot description, xacro)
@@ -48,5 +48,5 @@
         <origin xyz="0.0 0.0 0.0" rpy="0 0 ${pi*rotated}"/>
         <geometry>
-          <mesh filename="package://rfl/meshes/visual/${group}_z_axis_inner.stl"/>
+          <mesh filename="package://rfl/meshes/visual/${group}_z_axis.stl"/>
         </geometry>
         <xacro:material_abb_white />
@@ -55,5 +55,5 @@
         <origin xyz="0.0 0.0 0.0" rpy="0 0 ${pi*rotated}"/>
         <geometry>
-          <mesh filename="package://rfl/meshes/collision/${group}_z_axis_inner.stl"/>
+          <mesh filename="package://rfl/meshes/collision/${group}_z_axis.stl"/>
         </geometry>
       </collision>
@@ -67,34 +67,4 @@
     <!-- robot  -->
     <xacro:abb_irb4600_40_255 prefix="${prefix}_"/>
-    <!-- outer Z axis  -->
-    <joint name="${prefix}_joint_EA_Z_outer" type="prismatic">
-      <parent link="${prefix}_base"/>
-      <child link="${prefix}_z_axis_outer"/>
-      <origin xyz="0 0 0" rpy="0 0 0 "/>
-      <axis xyz="0 0 -1"/>
-      <limit lower="-10" upper="10" effort="100000" velocity="2.618" />
-      <dynamics damping="0.2" friction="0" />
-      <mimic joint="${prefix}_joint_EA_Z" multiplier="-0.5" offset="-2.4575" />
-    </joint>
-    <link name="${prefix}_z_axis_outer">
-      <inertial>
-        <origin xyz="0.0 0.0 0.0"/>
-        <mass value="120.00000"/>
-        <inertia ixx="-4.98000" iyy="-5.95200" izz="0.82800" ixy="-0.00000" ixz="2.70000" iyz="-0.00000"/>
-      </inertial>
-      <visual>
-        <origin xyz="0.0 0.0 0.0" rpy="0 0 ${pi*rotated}"/>
-        <geometry>
-          <mesh filename="package://rfl/meshes/visual/${group}_z_axis_outer.stl"/>
-        </geometry>
-        <xacro:material_abb_white />
-      </visual>
-      <collision>
-        <origin xyz="0.0 0.0 0.0" rpy="0 0 ${pi*rotated}"/>
-        <geometry>
-          <mesh filename="package://rfl/meshes/collision/${group}_z_axis_outer.stl"/>
-        </geometry>
-      </collision>
-    </link>
   </xacro:macro>
 </robot>

File: src/rfl/urdf/rfl.urdf (robot description, URDF)
Before this commit: robot rfl, 48 links, 47 joints
Links:
- removed link robot11_z_axis_outer
- removed link robot12_z_axis_outer
- removed link robot21_z_axis_outer
- removed link robot22_z_axis_outer
- link robot11_base: geometry collision mesh filename=package://rfl/meshes/collision/group1_z_axis.stl; visual mesh filename=package://rfl/meshes/visual/group1_z_axis.stl
- link robot12_base: geometry collision mesh filename=package://rfl/meshes/collision/group2_z_axis.stl; visual mesh filename=package://rfl/meshes/visual/group2_z_axis.stl
- link robot21_base: geometry collision mesh filename=package://rfl/meshes/collision/group2_z_axis.stl; visual mesh filename=package://rfl/meshes/visual/group2_z_axis.stl
- link robot22_base: geometry collision mesh filename=package://rfl/meshes/collision/group1_z_axis.stl; visual mesh filename=package://rfl/meshes/visual/group1_z_axis.stl
Joints:
- removed joint robot11_joint_EA_Z_outer
- removed joint robot12_joint_EA_Z_outer
- removed joint robot21_joint_EA_Z_outer
- removed joint robot22_joint_EA_Z_outer
