Commit message: package renaming inconsistency fix

File: rfl_description/urdf/bridge_macro.xacro (robot description, xacro)
@@ -20,5 +20,5 @@
         <origin xyz="0.0 ${12.2364997*rotated} 0.0" rpy="0 0 ${pi*rotated}"/>
         <geometry>
-          <mesh filename="package://rfl/meshes/visual/y_gantry.stl"/>
+          <mesh filename="package://rfl_description/meshes/visual/y_gantry.stl"/>
         </geometry>
         <xacro:material_abb_white/>
@@ -27,5 +27,5 @@
         <origin xyz="0.0 ${12.2364997*rotated} 0.0" rpy="0 0 ${pi*rotated}"/>
         <geometry>
-          <mesh filename="package://rfl/meshes/collision/y_gantry.stl"/>
+          <mesh filename="package://rfl_description/meshes/collision/y_gantry.stl"/>
         </geometry>
       </collision>

File: rfl_description/urdf/cart_macro.xacro (robot description, xacro)
@@ -20,5 +20,5 @@
         <origin xyz="0.0 0.0 0.0" rpy="0 0 ${pi*rotated}"/>
         <geometry>
-          <mesh filename="package://rfl/meshes/visual/${group}_xy_cart.stl"/>
+          <mesh filename="package://rfl_description/meshes/visual/${group}_xy_cart.stl"/>
         </geometry>
         <xacro:material_abb_white />
@@ -27,5 +27,5 @@
         <origin xyz="0.0 0.0 0.0" rpy="0 0 ${pi*rotated}"/>
         <geometry>
-          <mesh filename="package://rfl/meshes/collision/${group}_xy_cart.stl"/>
+          <mesh filename="package://rfl_description/meshes/collision/${group}_xy_cart.stl"/>
         </geometry>
       </collision>
@@ -48,5 +48,5 @@
         <origin xyz="0.0 0.0 0.0" rpy="0 0 ${pi*rotated}"/>
         <geometry>
-          <mesh filename="package://rfl/meshes/visual/${group}_z_axis_inner.stl"/>
+          <mesh filename="package://rfl_description/meshes/visual/${group}_z_axis_inner.stl"/>
         </geometry>
         <xacro:material_abb_white />
@@ -55,5 +55,5 @@
         <origin xyz="0.0 0.0 0.0" rpy="0 0 ${pi*rotated}"/>
         <geometry>
-          <mesh filename="package://rfl/meshes/collision/${group}_z_axis_inner.stl"/>
+          <mesh filename="package://rfl_description/meshes/collision/${group}_z_axis_inner.stl"/>
         </geometry>
       </collision>
@@ -86,5 +86,5 @@
         <origin xyz="0.0 0.0 0.0" rpy="0 0 ${pi*rotated}"/>
         <geometry>
-          <mesh filename="package://rfl/meshes/visual/${group}_z_axis_outer.stl"/>
+          <mesh filename="package://rfl_description/meshes/visual/${group}_z_axis_outer.stl"/>
         </geometry>
         <xacro:material_abb_white />
@@ -93,5 +93,5 @@
         <origin xyz="0.0 0.0 0.0" rpy="0 0 ${pi*rotated}"/>
         <geometry>
-          <mesh filename="package://rfl/meshes/collision/${group}_z_axis_outer.stl"/>
+          <mesh filename="package://rfl_description/meshes/collision/${group}_z_axis_outer.stl"/>
         </geometry>
       </collision>

File: rfl_description/urdf/rfl.urdf (robot description, URDF)
Before this commit: robot rfl, 48 links, 47 joints
Links:
- link bridge1: geometry collision mesh filename=package://rfl_description/meshes/collision/y_gantry.stl; visual mesh filename=package://rfl_description/meshes/visual/y_gantry.stl
- link bridge2: geometry collision mesh filename=package://rfl_description/meshes/collision/y_gantry.stl; visual mesh filename=package://rfl_description/meshes/visual/y_gantry.stl
- link robot11_base: geometry collision mesh filename=package://rfl_description/meshes/collision/group1_z_axis_in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; visual mesh filename=package://rfl_description/meshes/visual/group1_z_axis_inner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
- link robot11_xy_cart: geometry collision mesh filename=package://rfl_description/meshes/collision/group1_xy_cart.s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; visual mesh filename=package://rfl_description/meshes/visual/group1_xy_cart.stl
- link robot11_z_axis_outer: geometry collision mesh filename=package://rfl_description/meshes/collision/group1_z_axis_ou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; visual mesh filename=package://rfl_description/meshes/visual/group1_z_axis_outer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
- link robot12_base: geometry collision mesh filename=package://rfl_description/meshes/collision/group2_z_axis_in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; visual mesh filename=package://rfl_description/meshes/visual/group2_z_axis_inner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
- link robot12_xy_cart: geometry collision mesh filename=package://rfl_description/meshes/collision/group2_xy_cart.s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; visual mesh filename=package://rfl_description/meshes/visual/group2_xy_cart.stl
- link robot12_z_axis_outer: geometry collision mesh filename=package://rfl_description/meshes/collision/group2_z_axis_ou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; visual mesh filename=package://rfl_description/meshes/visual/group2_z_axis_outer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
- link robot21_base: geometry collision mesh filename=package://rfl_description/meshes/collision/group2_z_axis_in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; visual mesh filename=package://rfl_description/meshes/visual/group2_z_axis_inner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
- link robot21_xy_cart: geometry collision mesh filename=package://rfl_description/meshes/collision/group2_xy_cart.s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; visual mesh filename=package://rfl_description/meshes/visual/group2_xy_cart.stl
- link robot21_z_axis_outer: geometry collision mesh filename=package://rfl_description/meshes/collision/group2_z_axis_ou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; visual mesh filename=package://rfl_description/meshes/visual/group2_z_axis_outer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
- link robot22_base: geometry collision mesh filename=package://rfl_description/meshes/collision/group1_z_axis_in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; visual mesh filename=package://rfl_description/meshes/visual/group1_z_axis_inner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
- link robot22_xy_cart: geometry collision mesh filename=package://rfl_description/meshes/collision/group1_xy_cart.s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; visual mesh filename=package://rfl_description/meshes/visual/group1_xy_cart.stl
- link robot22_z_axis_outer: geometry collision mesh filename=package://rfl_description/meshes/collision/group1_z_axis_ou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; visual mesh filename=package://rfl_description/meshes/visual/group1_z_axis_outer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
- link world: geometry collision mesh filename=package://rfl_description/meshes/collision/rfl_floor_and_co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
- link x_rail: geometry collision mesh filename=package://rfl_description/meshes/collision/x_rail.stl; visual mesh filename=package://rfl_description/meshes/visual/x_rail.stl

File: rfl_description/urdf/rfl.xacro (robot description, xacro)
@@ -2,6 +2,6 @@
   xmlns:xacro="http://ros.org/wiki/xacro">
   <xacro:include filename="$(find abb_resources)/urdf/common_materials.xacro"/>
-  <xacro:include filename="$(find rfl)/urdf/bridge_macro.xacro"/>
-  <xacro:include filename="$(find rfl)/urdf/cart_macro.xacro"/>
+  <xacro:include filename="$(find rfl_description)/urdf/bridge_macro.xacro"/>
+  <xacro:include filename="$(find rfl_description)/urdf/cart_macro.xacro"/>
   <xacro:include filename="$(find abb_irb4600_40_255)/urdf/abb_irb4600_40_255_macro.xacro"/>
   <link name="world">
@@ -9,5 +9,5 @@
       <origin xyz="0.0 0.0 0.0" rpy="0.0 0.0 0.0"/>
       <geometry>
-        <mesh filename="package://rfl/meshes/collision/rfl_floor_and_columns.stl"/>
+        <mesh filename="package://rfl_description/meshes/collision/rfl_floor_and_columns.stl"/>
       </geometry>
     </collision>
@@ -22,5 +22,5 @@
       <origin xyz="0 0 0" rpy="0 0 0"/>
       <geometry>
-        <mesh filename="package://rfl/meshes/visual/x_rail.stl"/>
+        <mesh filename="package://rfl_description/meshes/visual/x_rail.stl"/>
       </geometry>
       <xacro:material_abb_white/>
@@ -29,5 +29,5 @@
       <origin xyz="0 0 0" rpy="0 0 0"/>
       <geometry>
-        <mesh filename="package://rfl/meshes/collision/x_rail.stl"/>
+        <mesh filename="package://rfl_description/meshes/collision/x_rail.stl"/>
       </geometry>
     </collision>
