Commit message: package renaming inconsistency fix

File: rfl_description/urdf/cart_macro.xacro (robot description, xacro)
@@ -20,5 +20,5 @@
         <origin xyz="0.0 0.0 0.0" rpy="0 0 ${pi*rotated}"/>
         <geometry>
-          <mesh filename="package://rfl/meshes/visual/${group}_xy_cart.stl"/>
+          <mesh filename="package://rfl_description/meshes/visual/${group}_xy_cart.stl"/>
         </geometry>
         <xacro:material_abb_white />
@@ -27,5 +27,5 @@
         <origin xyz="0.0 0.0 0.0" rpy="0 0 ${pi*rotated}"/>
         <geometry>
-          <mesh filename="package://rfl/meshes/collision/${group}_xy_cart.stl"/>
+          <mesh filename="package://rfl_description/meshes/collision/${group}_xy_cart.stl"/>
         </geometry>
       </collision>
@@ -48,5 +48,5 @@
         <origin xyz="0.0 0.0 0.0" rpy="0 0 ${pi*rotated}"/>
         <geometry>
-          <mesh filename="package://rfl/meshes/visual/${group}_z_axis.stl"/>
+          <mesh filename="package://rfl_description/meshes/visual/${group}_z_axis.stl"/>
         </geometry>
         <xacro:material_abb_white />
@@ -55,5 +55,5 @@
         <origin xyz="0.0 0.0 0.0" rpy="0 0 ${pi*rotated}"/>
         <geometry>
-          <mesh filename="package://rfl/meshes/collision/${group}_z_axis.stl"/>
+          <mesh filename="package://rfl_description/meshes/collision/${group}_z_axis.stl"/>
         </geometry>
       </collision>

File: rfl_description/urdf/rfl.urdf (robot description, URDF)
Before this commit: robot rfl, 44 links, 43 joints
Links:
- link bridge1: geometry collision mesh filename=package://rfl_description/meshes/collision/y_gantry.stl; visual mesh filename=package://rfl_description/meshes/visual/y_gantry.stl
- link bridge2: geometry collision mesh filename=package://rfl_description/meshes/collision/y_gantry.stl; visual mesh filename=package://rfl_description/meshes/visual/y_gantry.stl
- link robot11_base: geometry collision mesh filename=package://rfl_description/meshes/collision/group1_z_axis.stl; visual mesh filename=package://rfl_description/meshes/visual/group1_z_axis.stl
- link robot11_xy_cart: geometry collision mesh filename=package://rfl_description/meshes/collision/group1_xy_cart.s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; visual mesh filename=package://rfl_description/meshes/visual/group1_xy_cart.stl
- link robot12_base: geometry collision mesh filename=package://rfl_description/meshes/collision/group2_z_axis.stl; visual mesh filename=package://rfl_description/meshes/visual/group2_z_axis.stl
- link robot12_xy_cart: geometry collision mesh filename=package://rfl_description/meshes/collision/group2_xy_cart.s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; visual mesh filename=package://rfl_description/meshes/visual/group2_xy_cart.stl
- link robot21_base: geometry collision mesh filename=package://rfl_description/meshes/collision/group2_z_axis.stl; visual mesh filename=package://rfl_description/meshes/visual/group2_z_axis.stl
- link robot21_xy_cart: geometry collision mesh filename=package://rfl_description/meshes/collision/group2_xy_cart.s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; visual mesh filename=package://rfl_description/meshes/visual/group2_xy_cart.stl
- link robot22_base: geometry collision mesh filename=package://rfl_description/meshes/collision/group1_z_axis.stl; visual mesh filename=package://rfl_description/meshes/visual/group1_z_axis.stl
- link robot22_xy_cart: geometry collision mesh filename=package://rfl_description/meshes/collision/group1_xy_cart.s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; visual mesh filename=package://rfl_description/meshes/visual/group1_xy_cart.stl
- link world: geometry collision mesh filename=package://rfl_description/meshes/collision/rfl_floor_and_co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
- link x_rail: geometry collision mesh filename=package://rfl_description/meshes/collision/x_rail.stl; visual mesh filename=package://rfl_description/meshes/visual/x_rail.stl
