Commit message: adding rfl_floor_and_columns.stl visual mesh to URDF

File: rfl_description/urdf/rfl.xacro (robot description, xacro)
@@ -6,4 +6,10 @@
   <xacro:include filename="$(find abb_irb4600_40_255)/urdf/abb_irb4600_40_255_macro.xacro"/>
   <link name="world">
+  <visual>
+      <origin rpy="0.0 0.0 0.0" xyz="0.0 0.0 0.0"/>
+      <geometry>
+        <mesh filename="package://rfl_description/meshes/visual/rfl_floor_and_columns.stl"/>
+      </geometry>
+    </visual>
     <collision>
       <origin xyz="0.0 0.0 0.0" rpy="0.0 0.0 0.0"/>

Commit message: indentation fix

File: rfl_description/urdf/rfl.xacro (robot description, xacro)
@@ -6,5 +6,5 @@
   <xacro:include filename="$(find abb_irb4600_40_255)/urdf/abb_irb4600_40_255_macro.xacro"/>
   <link name="world">
-  <visual>
+    <visual>
       <origin rpy="0.0 0.0 0.0" xyz="0.0 0.0 0.0"/>
       <geometry>
