Commit message: xacro-urdf update to include rfl_floor_and_columns visual mesh

File: rfl_description/urdf/rfl.urdf (robot description, URDF)
Before this commit: robot rfl, 44 links, 43 joints
Links:
- link world: geometry collision mesh filename=package://rfl_description/meshes/collision/rfl_floor_and_co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; visual mesh filename=package://rfl_description/meshes/visual/rfl_floor_and_colum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

Commit message: adjusting ABB arm joint 4 + 5 length

File: rfl_description/urdf/rfl.urdf (robot description, URDF)
Before this commit: robot rfl, 44 links, 43 joints
Joints:
- joint robot11_joint_4: origin xyz=0.332 0 0.175 rpy=0 0 0  -> xyz=0.331 0 0.175 rpy=0 0 0 
- joint robot12_joint_4: origin xyz=0.332 0 0.175 rpy=0 0 0  -> xyz=0.331 0 0.175 rpy=0 0 0 
- joint robot21_joint_4: origin xyz=0.332 0 0.175 rpy=0 0 0  -> xyz=0.331 0 0.175 rpy=0 0 0 
- joint robot22_joint_4: origin xyz=0.332 0 0.175 rpy=0 0 0  -> xyz=0.331 0 0.175 rpy=0 0 0 
